Commit message: adjust car properties and move baselink

File: src/car_simulator/models/race_car/model.urdf (robot description, URDF)
Before this commit: robot sam_bot, 6 links, 5 joints
Joints:
- joint base_link_joint: origin xyz=${-base_x_origin_to_wheel_origin} 0 0.05 rpy=0 0 0 -> xyz=${base_x_origin_to_wheel_origin-0.01} 0 0.05 rpy=0 0 0
